File: monocam_hat.kicad_pcb (KiCad board)
At the start: 2 copper layers, 56.6 x 18.8 mm, 27 parts, among them J1 Conn_02x20_Odd_Even, U1 LM3671MF-2.8, U2 OV7690, U3 TXS0102DCT, U4 ASDMB-xxxMHz, U5 74LV8T245, U6 74LV8T245, U7 L3GD20

Commit message: V2 layout complete
Parts:
- added C13: 10uF, Capacitor_SMD:C_0402_1005Metric, F.Cu at (214.1, 109.8)
- L1, L2, L3: footprint Inductor_SMD:L_0402_1005Metric -> Inductor_SMD:L_0603_1608Metric
- moved L3 1.19 mm to (221.8, 101.9), turned to 180 degrees
- moved C5 0.56 mm to (218.3, 102.1)
- moved C3 0.25 mm to (215.6, 104.6)
- moved C2 0.25 mm to (216.8, 104.6)
- moved L1 0.15 mm to (218.2, 104.6)
Routing:
- net GND: track 33.2 -> 35.2 mm
- net Net-(C11-Pad2): track 3.08 -> 4.25 mm
- net +2V8: track 7.09 -> 6.08 mm
- net VDDA: track 26.4 -> 26.9 mm
