File: monocam_hat.sch (KiCad schematic (older format))
At the start: 28 parts, among them J1 Conn_02x20_Odd_Even, U1 LM3671MF-2.8, U2 OV7690, U3 TXS0102DCT, U4 ASDMB-xxxMHz, U5 74LV8T245, U6 74LV8T245, U7 L3GD20

Commit message: V2 layout complete
Parts:
- L1, L2, L3: footprint Inductor_SMD:L_0402_1005Metric -> Inductor_SMD:L_0603_1608Metric
- gave numbers to parts that had none: 1
Changed lines of the file:
@@
 F 0 "L2" V 2485 6900 50  0000 C CNN
 F 1 "2.2uH" V 2394 6900 50  0000 C CNN
-F 2 "Inductor_SMD:L_0402_1005Metric" H 2300 6900 50  0001 C CNN
+F 2 "Inductor_SMD:L_0603_1608Metric" H 2300 6900 50  0001 C CNN
 F 3 "~" H 2300 6900 50  0001 C CNN
 	1    2300 6900
@@
 F 0 "L3" V 2590 5800 50  0000 C CNN
 F 1 "3.3uH" V 2499 5800 50  0000 C CNN
-F 2 "Inductor_SMD:L_0402_1005Metric" H 2400 5800 50  0001 C CNN
+F 2 "Inductor_SMD:L_0603_1608Metric" H 2400 5800 50  0001 C CNN
 F 3 "~" H 2400 5800 50  0001 C CNN
 	1    2400 5800
@@
 F 0 "L1" V 1940 5750 50  0000 C CNN
 F 1 "3.3uH" V 1849 5750 50  0000 C CNN
-F 2 "Inductor_SMD:L_0402_1005Metric" H 1750 5750 50  0001 C CNN
+F 2 "Inductor_SMD:L_0603_1608Metric" H 1750 5750 50  0001 C CNN
 F 3 "~" H 1750 5750 50  0001 C CNN
 	1    1750 5750
@@
 $EndComp
 $Comp
-L power:GND #PWR?
+L power:GND #PWR0143
 U 1 1 5F58CC8D
 P 2050 2900
-F 0 "#PWR?" H 2050 2650 50  0001 C CNN
+F 0 "#PWR0143" H 2050 2650 50  0001 C CNN
 F 1 "GND" V 2055 2772 50  0000 R CNN
 F 2 "" H 2050 2900 50  0001 C CNN
@@
 $EndComp
 $Comp
-L power:GND #PWR?
+L power:GND #PWR0144
 U 1 1 5F58E811
 P 2050 3300
-F 0 "#PWR?" H 2050 3050 50  0001 C CNN
+F 0 "#PWR0144" H 2050 3050 50  0001 C CNN
 F 1 "GND" V 2055 3172 50  0000 R CNN
 F 2 "" H 2050 3300 50  0001 C CNN
@@
 $EndComp
 $Comp
-L power:GND #PWR?
+L power:GND #PWR0145
 U 1 1 5F5950A4
 P 2050 3700
-F 0 "#PWR?" H 2050 3450 50  0001 C CNN
+F 0 "#PWR0145" H 2050 3450 50  0001 C CNN
 F 1 "GND" V 2055 3572 50  0000 R CNN
 F 2 "" H 2050 3700 50  0001 C CNN
@@
 $EndComp
 $Comp
-L power:GND #PWR?
+L power:GND #PWR0146
 U 1 1 5F59B98C
 P 2050 4100
-F 0 "#PWR?" H 2050 3850 50  0001 C CNN
+F 0 "#PWR0146" H 2050 3850 50  0001 C CNN
 F 1 "GND" V 2055 3972 50  0000 R CNN
 F 2 "" H 2050 4100 50  0001 C CNN
@@
 $EndComp
 $Comp
-L power:GND #PWR?
+L power:GND #PWR0147
 U 1 1 5F5A2E8C
 P 2750 2900
-F 0 "#PWR?" H 2750 2650 50  0001 C CNN
+F 0 "#PWR0147" H 2750 2650 50  0001 C CNN
 F 1 "GND" V 2755 2772 50  0000 R CNN
 F 2 "" H 2750 2900 50  0001 C CNN
@@
 $EndComp
 $Comp
-L power:GND #PWR?
+L power:GND #PWR0148
 U 1 1 5F5A95E2
 P 2750 3300
-F 0 "#PWR?" H 2750 3050 50  0001 C CNN
+F 0 "#PWR0148" H 2750 3050 50  0001 C CNN
 F 1 "GND" V 2755 3172 50  0000 R CNN
 F 2 "" H 2750 3300 50  0001 C CNN
@@
 $EndComp
 $Comp
-L power:GND #PWR?
+L power:GND #PWR0149
 U 1 1 5F5AFCB4
 P 2750 3700
-F 0 "#PWR?" H 2750 3450 50  0001 C CNN
+F 0 "#PWR0149" H 2750 3450 50  0001 C CNN
 F 1 "GND" V 2755 3572 50  0000 R CNN
 F 2 "" H 2750 3700 50  0001 C CNN
@@
 $EndComp
 $Comp
-L power:GND #PWR?
+L power:GND #PWR0150
 U 1 1 5F5B639C
 P 2750 4100
-F 0 "#PWR?" H 2750 3850 50  0001 C CNN
+F 0 "#PWR0150" H 2750 3850 50  0001 C CNN
 F 1 "GND" V 2755 3972 50  0000 R CNN
 F 2 "" H 2750 4100 50  0001 C CNN
@@
 $EndComp
 $Comp
-L Device:C_Small C?
+L Device:C_Small C13
 U 1 1 5F52F7EA
 P 3950 3400
-F 0 "C?" H 4042 3446 50  0000 L CNN
+F 0 "C13" H 4042 3446 50  0000 L CNN
 F 1 "10uF" H 4042 3355 50  0000 L CNN
 F 2 "Capacitor_SMD:C_0402_1005Metric" H 3950 3400 50  0001 C CNN
